File: br2_5v_interface_U_starter.kicad_sch (KiCad schematic)
At the start: 18 parts, among them J10 BR2_BANK_A_J10, J11 BR2_BANK_B_J11, J12 BR2_BANK_B_J12, J13 BR2_BANK_B_J13, J14 BR2_BANK_B_J14, J17 BR2_CONTROL_J17, J18 BR2_CONTROL_J18, J19 BR2_CONTROL_J19, J20 BR2_CONTROL_J20, J21 5V_OUTPUTS_U1, J7 BR2_BANK_A_J7, J8 BR2_BANK_A_J8, J9 BR2_BANK _A_J9, U1 SN74AHCT245N

Commit message: Mac version: align BR2 headers and update PCB routing
Connections:
- net +5V: now also J20.1 (Pin_1)
- no-connect marks 136 -> 135

Commit message: Correct 5V and 3.3V connections
Connections:
- net +5V: now also J19.1 (Pin_1); no longer J20.1 (Pin_1)
- new net +3.3vdc: J20.1 (Pin_1)
- no-connect marks 135 -> 134
Changed lines of the file:
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@@
+	)
+	(no_connect
+		(at 30.48 50.8)
+	)
+	(no_connect
+		(at 82.55 90.17)
+	)
+	(no_connect
+		(at 50.8 146.05)
+	)
+	(no_connect
+		(at 30.48 45.72)
+	)
+	(no_connect
+		(at 110.49 33.02)
+	)
+	(no_connect
+		(at 30.48 116.84)
+	)
+	(no_connect
+		(at 30.48 38.1)
+	)
+	(no_connect
+		(at 110.49 38.1)
+	)
+	(no_connect
+		(at 30.48 140.97)
+	)
+	(no_connect
+		(at 30.48 114.3)
+	)
+	(no_connect
+		(at 255.27 66.04)
+	)
+	(no_connect
+		(at 110.49 69.85)
+	)
+	(no_connect
+		(at 54.61 74.93)
+	)
+	(no_connect
+		(at 50.8 143.51)
+	)
+	(no_connect
+		(at 82.55 53.34)
+	)
+	(no_connect
+		(at 82.55 80.01)
+	)
+	(no_connect
+		(at 30.48 127)
+	)
+	(no_connect
+		(at 50.8 121.92)
+	)
+	(no_connect
+		(at 54.61 90.17)
+	)
+	(no_connect
+		(at 82.55 43.18)
+	)
+	(no_connect
+		(at 255.27 63.5)
+	)
+	(no_connect
+		(at 54.61 82.55)
+	)
+	(no_connect
+		(at 82.55 40.64)
+	)
+	(no_connect
+		(at 54.61 69.85)
+	)
+	(no_connect
+		(at 54.61 22.86)
+	)
+	(no_connect
+		(at 110.49 74.93)
+	)
+	(no_connect
+		(at 30.48 97.79)
+	)
+	(no_connect
+		(at 30.48 25.4)
+	)
+	(no_connect
+		(at 82.55 97.79)
+	)
+	(no_connect
+		(at 82.55 100.33)
+	)
+	(no_connect
+		(at 30.48 82.55)
+	)
+	(no_connect
+		(at 110.49 48.26)
+	)
+	(no_connect
+		(at 82.55 30.48)
+	)
+	(no_connect
+		(at 54.61 55.88)
+	)
+	(no_connect
+		(at 110.49 30.48)
+	)
+	(no_connect
+		(at 54.61 33.02)
+	)
+	(no_connect
+		(at 82.55 27.94)
+	)
+	(no_connect
+		(at 82.55 95.25)
+	)
+	(no_connect
+		(at 82.55 38.1)
+	)
+	(no_connect
+		(at 110.49 100.33)
+	)
+	(no_connect
+		(at 54.61 97.79)
+	)
+	(no_connect
+		(at 110.49 92.71)
+	)
+	(no_connect
+		(at 82.55 45.72)
+	)
+	(no_connect
+		(at 30.48 27.94)
+	)
+	(no_connect
+		(at 30.48 74.93)
+	)
+	(no_connect
+		(at 82.55 35.56)
+	)
+	(no_connect
+		(at 30.48 151.13)
+	)
+	(no_connect
+		(at 213.36 63.5)
+	)
+	(no_connect
+		(at 82.55 48.26)
 	)
 	(no_connect
@@
 	)
 	(no_connect
-		(at 30.48 50.8)
-	)
-	(no_connect
-		(at 82.55 90.17)
-	)
-	(no_connect
-		(at 50.8 146.05)
-	)
-	(no_connect
-		(at 30.48 45.72)
-	)
-	(no_connect
-		(at 110.49 33.02)
-	)
-	(no_connect
-		(at 30.48 116.84)
-	)
-	(no_connect
-		(at 30.48 38.1)
-	)
-	(no_connect
-		(at 110.49 38.1)
-	)
-	(no_connect
-		(at 30.48 114.3)
-	)
-	(no_connect
-		(at 255.27 66.04)
-	)
-	(no_connect
-		(at 110.49 69.85)
-	)
-	(no_connect
-		(at 54.61 74.93)
-	)
-	(no_connect
-		(at 50.8 143.51)
-	)
-	(no_connect
-		(at 82.55 53.34)
-	)
-	(no_connect
-		(at 82.55 80.01)
-	)
-	(no_connect
-		(at 30.48 127)
-	)
-	(no_connect
-		(at 50.8 121.92)
-	)
-	(no_connect
-		(at 54.61 90.17)
-	)
-	(no_connect
-		(at 82.55 43.18)
-	)
-	(no_connect
-		(at 255.27 63.5)
-	)
-	(no_connect
-		(at 54.61 82.55)
-	)
-	(no_connect
-		(at 82.55 40.64)
-	)
-	(no_connect
-		(at 54.61 69.85)
-	)
-	(no_connect
-		(at 54.61 22.86)
-	)
-	(no_connect
-		(at 110.49 74.93)
-	)
-	(no_connect
-		(at 30.48 97.79)
-	)
-	(no_connect
-		(at 30.48 25.4)
-	)
-	(no_connect
-		(at 82.55 97.79)
-	)
-	(no_connect
-		(at 82.55 100.33)
-	)
-	(no_connect
-		(at 30.48 82.55)
-	)
-	(no_connect
-		(at 110.49 48.26)
-	)
-	(no_connect
-		(at 82.55 30.48)
-	)
-	(no_connect
-		(at 54.61 55.88)
-	)
-	(no_connect
-		(at 110.49 30.48)
-	)
-	(no_connect
-		(at 54.61 33.02)
-	)
-	(no_connect
-		(at 82.55 27.94)
-	)
-	(no_connect
-		(at 82.55 95.25)
-	)
-	(no_connect
-		(at 82.55 38.1)
-	)
-	(no_connect
-		(at 110.49 100.33)
-	)
-	(no_connect
-		(at 54.61 97.79)
-	)
-	(no_connect
-		(at 110.49 92.71)
-	)
-	(no_connect
-		(at 82.55 45.72)
-	)
-	(no_connect
-		(at 30.48 27.94)
-	)
-	(no_connect
-		(at 30.48 74.93)
-	)
-	(no_connect
-		(at 82.55 35.56)
-	)
-	(no_connect
-		(at 30.48 151.13)
-	)
-	(no_connect
-		(at 213.36 63.5)
-	)
-	(no_connect
-		(at 82.55 48.26)
-	)
-	(no_connect
 		(at 82.55 25.4)
 	)
@@
 	)
 	(no_connect
-		(at 30.48 140.97)
-	)
-	(no_connect
 		(at 110.49 85.09)
 	)
@@
 	)
 	(no_connect
-		(at 30.48 138.43)
-	)
-	(no_connect
 		(at 82.55 55.88)
 	)
@@
 		(pts
 			(xy 157.48 63.5) (xy 157.48 74.93)
+		)
+		(stroke
+			(width 0)
+			(type default)
+		)
+	)
+	(wire
+		(pts
+			(xy 30.48 138.43) (xy 33.02 138.43)
 		)
 		(stroke
@@
 				(path "/0e211f18-c279-46d1-80af-e05e6025d205"
 					(reference "#PWR05")
+					(unit 1)
+				)
+			)
+		)
+	)
+	(symbol
+		(lib_name "+5V_2")
+		(lib_id "power:+5V")
+		(at 33.02 138.43 270)
+		(unit 1)
+		(exclude_from_sim no)
+		(in_bom yes)
+		(on_board yes)
+		(dnp no)
+		(fields_autoplaced yes)
+		(property "Reference" "#PWR07"
+			(at 29.21 138.43 0)
+			(effects
+				(font
+					(size 1.27 1.27)
+				)
+				(hide yes)
+			)
+		)
+		(property "Value" "+5V"
+			(at 36.83 138.4299 90)
+			(effects
+				(font
+					(size 1.27 1.27)
+				)
+				(justify left)
+			)
+		)
+		(property "Footprint" ""
+			(at 33.02 138.43 0)
+			(effects
+				(font
+					(size 1.27 1.27)
+				)
+				(hide yes)
+			)
+		)
+		(property "Datasheet" ""
+			(at 33.02 138.43 0)
+			(effects
+				(font
+					(size 1.27 1.27)
+				)
+				(hide yes)
+			)
+		)
+		(property "Description" "Power symbol creates a global label with name \"+5V\""
+			(at 33.02 138.43 0)
+			(effects
+				(font
+					(size 1.27 1.27)
+				)
+				(hide yes)
+			)
+		)
+		(pin "1"
+		)
+		(instances
+			(project ""
+				(path "/0e211f18-c279-46d1-80af-e05e6025d205"
+					(reference "#PWR07")
 					(unit 1)
 				)
@@
 			)
 		)
-		(property "Value" "+5V"
-			(at 62.23 132.08 0)
-			(effects
-				(font
-					(size 1.27 1.27)
-				)
-			)
-		)
+		(property "Value" "+3.3vdc"
+			(at 64.77 135.8899 0)
+			(effects
+				(font
+					(size 1.27 1.27)
+				)
+				(justify left)
+			)
+		)

Commit message: Update BR2 interface PCB and schematic with corrected pin mappings
Connections:
- net B24_RAM_CS_N: now also J11.5 (Pin_5); no longer J14.5 (Pin_5)
- net B28_UART_B_CS_N: now also J12.5 (Pin_5); no longer J13.6 (Pin_6)
- net B30_ACIA_CS_N: now also J11.6 (Pin_6); no longer J14.6 (Pin_6)
- net B42_ROM_CS_N: now also J11.8 (Pin_8); no longer J14.8 (Pin_8)
Other:
- company: (none) -> SABE
- moved on the sheet: J10, J14, J9
